Commit message: Fully integrated end to end stack, mapping not yet working properly, LIDAR integrated with local map

File: src/rbcar_common-kinetic-devel/rbcar_description/robots/rbcar.urdf.xacro (robot description, xacro)
@@ -43,5 +43,5 @@
 	<!-- SENSORS -->
     <xacro:sensor_sick_s3000 prefix="front_laser" parent="base_link">
-		<origin xyz="1.58 0.0 0.0" rpy="0 0.0 0"/>
+		<origin xyz="1.58 0.0 0.5" rpy="0 0.0 0"/>
 	</xacro:sensor_sick_s3000>
 	<xacro:sensor_imu prefix="imu" parent="base_link">
