Commit message: Pushing navigation stack, in good shape

File: src/robotnik_sensors-kinetic-devel/urdf/sick_s3000.urdf.xacro (robot description, xacro)
@@ -26,5 +26,5 @@
 		</inertial>
 	</link>
-	<!-- Sick sensor sensor for simulation -->
+	<!-- Sick sensor sensor for simulation
 	<sensor_sick_s3000_gazebo/>
   </xacro:macro>
@@ -70,3 +70,48 @@
 	</gazebo>
   </xacro:macro>
+ -->
+<!-- Sick sensor sensor for simulation -->
+	<sensor_sick_s3000_gazebo/>
+  </xacro:macro>
+  <xacro:macro name="sensor_sick_s3000_gazebo">
+    <gazebo reference="${prefix}_base_link">
+		<xacro:if value="${gpu}">
+			<xacro:property name="ray_type" value="gpu_ray" />
+			<xacro:property name="plugin_lib" value="libgazebo_ros_gpu_laser.so" />
+		</xacro:if>
+		<xacro:unless value="${gpu}">
+			<xacro:property name="ray_type" value="ray" />
+			<xacro:property name="plugin_lib" value="libgazebo_ros_laser.so" />
+		</xacro:unless>
+		<sensor type="${ray_type}" name="${prefix}_sensor">
+			<pose>0 0 0 0 0 0</pose>
+			<visualize>false</visualize>
+			<update_rate>16.6</update_rate>
+			<ray>
+				<scan>
+					<horizontal>
+						<samples>761</samples>
+						<resolution>1</resolution>
+						<min_angle>-1.6580</min_angle>
+						<max_angle>1.6580</max_angle>
+					</horizontal>
+				</scan>
+				<range>
+					<min>0.10</min>
+					<max>100.0</max>
+					<resolution>0.01</resolution>
+				</range>
+				<noise>
+					<type>gaussian</type>
+					<mean>0.0</mean>
+					<stddev>0.0</stddev>
+				</noise>
+			</ray>
+			<plugin name="${prefix}_controller" filename="${plugin_lib}">
+				<topicName>${ns}${prefix_topic}/scan</topicName>
+				<frameName>/${prefix}_base_link</frameName>
+			</plugin>
+		</sensor>
+	</gazebo>
+  </xacro:macro>
 </robot>
